Commit message: modified:   movo_7dof_moveit_config/config/movo_kg2.srdf 	modified:   movo_7dof_moveit_config/config/movo_kg3.srdf 	modified:   movo_common/movo_description/urdf/sensors/kinect_one_sensor.urdf.xacro 	modified:   movo_servo_teleop_demo/config/fake_kinova_bridge.yaml 	modified:   movo_servo_teleop_demo/scripts/fake_kinova_command_bridge.py

File: movo_common/movo_description/urdf/sensors/kinect_one_sensor.urdf.xacro (robot description, xacro)
@@ -47,9 +47,4 @@
 				</geometry>
 			</visual>
-			<collision>
-				<geometry>
-					<mesh filename="package://movo_description/meshes/sensors/collision/kinect_one_collision.stl" />
-				</geometry>
-			</collision>
 		</link>
         <link name="${prefix}_ir_link"/>
