Commit message: modified:   movo_7dof_moveit_config/config/joint_limits.yaml 	modified:   movo_common/movo_description/urdf/movo.urdf.xacro 	modified:   movo_servo/config/left_arm_servo.yaml 	modified:   movo_servo/config/right_arm_servo.yaml 	modified:   movo_servo_teleop_demo/config/left_arm_servo.yaml 	modified:   movo_servo_teleop_demo/config/right_arm_servo.yaml

File: movo_common/movo_description/urdf/movo.urdf.xacro (robot description, xacro)
@@ -73,8 +73,8 @@
     		<xacro:include filename="$(find movo_description)/urdf/manipulation/jaco/jaco_7dof.urdf.xacro" />
             <xacro:jaco_robot_7dof prefix="right_" parent="linear_actuator_link">
-            <origin xyz="0.0261046 -0.13335 0.2799937" rpy="${-M_PI/2} 0 ${-M_PI/2}"/>
+            <origin xyz="0.0961046 -0.13335 0.2799937" rpy="${-M_PI/2} 0 ${-M_PI/2}"/>
             </xacro:jaco_robot_7dof>
             <xacro:jaco_robot_7dof prefix="left_" parent="linear_actuator_link">
-                <origin xyz="0.0261046 0.13335 0.2799937" rpy="${-M_PI/2} 0 ${-M_PI/2}"/>
+                <origin xyz="0.0961046 0.13335 0.2799937" rpy="${-M_PI/2} 0 ${-M_PI/2}"/>
             </xacro:jaco_robot_7dof>
         </xacro:if>
@@ -82,9 +82,9 @@
         	<xacro:include filename="$(find movo_description)/urdf/manipulation/jaco/jaco.urdf.xacro" />
             <xacro:jaco_robot prefix="right_" parent="linear_actuator_link">
-		        <origin xyz="0.0261046 -0.13335 0.2799937" rpy="${-M_PI/2} 0 ${-M_PI/2}"/>
+		        <origin xyz="0.0961046 -0.13335 0.2799937" rpy="${-M_PI/2} 0 ${-M_PI/2}"/>
 		    </xacro:jaco_robot>
 		    <xacro:if value="$(optenv MOVO_HAS_TWO_KINOVA_ARMS false)">
 		        <xacro:jaco_robot prefix="left_" parent="linear_actuator_link">
-		            <origin xyz="0.0261046 0.13335 0.2799937" rpy="${-M_PI/2} 0 ${-M_PI/2}"/>
+		            <origin xyz="0.0961046 0.13335 0.2799937" rpy="${-M_PI/2} 0 ${-M_PI/2}"/>
 		        </xacro:jaco_robot>
 		    </xacro:if>
